File: big7segment/big7segment.brd (EAGLE design)
At the start: 90 x 122 mm, 48 parts

Commit message: new desing and simulate 7 segment
Parts:
- removed LED10, LED11, LED12, LED13, LED14, LED15, LED16, LED17, LED18, LED19, LED20, LED21, LED22, LED7, LED8, LED9: (no value), led:SML0805
- added B1, B2, B3, B4, C1, C2, C3, C4, C5, D1, D2, D3, D4, D5, D6, DOT1, DOT2, DOT3, DOT4, E1, E2, E3, E4, E5, F1, F2, F3, F4, F5, G1, G2, G3, G4, G5, G6: (no value), led:SML0805
- added JP1: (no value), SparkFun-Jumpers:SMT-JUMPER_2_NC_TRACE_NO-SILK
- added JP2: (no value), SparkFun-Jumpers:SMT-JUMPER_2_NO_NO-SILK
- added Q1, Q10, Q12, Q14, Q16, Q18, Q4, Q6, Q8: NMOS, SparkFun-DiscreteSemi:SOT23-3
- added Q11, Q13, Q15, Q17, Q2, Q3, Q5, Q7, Q9: PMOS, SparkFun-DiscreteSemi:SOT23-3
- added R1, R10, R11, R12, R13, R14, R15, R16, R17, R18, R19, R2, R20, R21, R22, R23, R24, R25, R26, R27, R28, R29, R3, R30, R31, R32, R33, R34, R35, R36, R37, R38, R39, R4, R40, R41, R42, R5, R6, R7, R8, R9: 180, SparkFun-Resistors:0805
- added R43, R44, R47, R48, R49, R51, R52, R54, R55, R57, R58, R60, R61, R63, R64, R66, R67, R69: 10k, SparkFun-Resistors:0805
- added R45, R46, R50, R53, R56, R59, R62, R65, R68: 4.7k, SparkFun-Resistors:0805
- renumbered + to 5V, COM to !ENABLE!, LED1 to A1, LED2 to A2, LED23 to B5, LED3 to A3, LED4 to A4, LED5 to A5, LED6 to A6
Connections:
- new net !ENABLE!: !ENABLE!.1, JP2.1, R46.2
- new net COMMON: A1.C, A2.C, A3.C, A4.C, A5.C, A6.C, B1.C, B2.C, B3.C, B4.C, B5.C, C1.C, C2.C, C3.C, C4.C, C5.C, D1.C, D2.C, D3.C, D4.C, D5.C, D6.C, DOT1.C, DOT2.C, DOT3.C, DOT4.C, E1.C, E2.C, E3.C, E4.C, E5.C, F1.C, F2.C, F3.C, F4.C, F5.C, G1.C, G2.C, G3.C, G4.C, G5.C, G6.C, Q4.3
- new net N$1: A1.A, R1.1
- new net N$10: B4.A, R10.1
- new net N$11: B5.A, R11.1
- new net N$12: C1.A, R12.1
- new net N$13: C2.A, R13.1
- new net N$14: C3.A, R14.1
- new net N$15: C4.A, R15.1
- new net N$16: C5.A, R16.1
- new net N$17: D1.A, R17.1
- new net N$18: D2.A, R18.1
- new net N$19: D3.A, R19.1
- new net N$2: A3.A, R3.1
- new net N$20: D4.A, R20.1
- new net N$21: D5.A, R21.1
- new net N$22: D6.A, R22.1
- new net N$23: E1.A, R23.1
- new net N$24: E2.A, R24.1
- new net N$25: E3.A, R25.1
- new net N$26: E4.A, R26.1
- new net N$27: E5.A, R27.1
- new net N$28: F1.A, R28.1
- new net N$29: F2.A, R29.1
- new net N$3: A4.A, R4.1
- new net N$30: F3.A, R30.1
- new net N$31: F4.A, R31.1
- new net N$32: F5.A, R32.1
- new net N$33: G1.A, R33.1
- new net N$34: G2.A, R34.1
- new net N$35: G3.A, R35.1
- new net N$36: G4.A, R36.1
- new net N$37: G5.A, R37.1
- new net N$38: G6.A, R38.1
- new net N$39: DOT1.A, R39.1
- new net N$4: A5.A, R5.1
- new net N$40: DOT2.A, R40.1
- new net N$41: DOT3.A, R41.1
- new net N$42: DOT4.A, R42.1
- new net N$43: Q2.1, R44.1, R45.2
- new net N$44: Q1.3, R45.1
- new net N$45: Q5.1, R49.1, R50.2
- new net N$46: Q2.3, R1.2, R2.2, R3.2, R4.2, R5.2, R6.2
- new net N$47: Q3.1, R46.1, R47.1
- new net N$48: JP2.2, Q3.3, Q4.1, R48.2
- new net N$49: Q5.3, R10.2, R11.2, R7.2, R8.2, R9.2
- new net N$5: A6.A, R6.1
- new net N$50: Q11.1, R58.1, R59.2
- new net N$51: Q12.3, R59.1
- new net N$52: Q6.3, R50.1
- new net N$53: Q7.1, R52.1, R53.2
- new net N$54: Q8.3, R53.1
- new net N$55: Q7.3, R12.2, R13.2, R14.2, R15.2, R16.2
- new net N$56: Q9.1, R55.1, R56.2
- new net N$57: Q10.3, R56.1
- new net N$58: Q9.3, R17.2, R18.2, R19.2, R20.2, R21.2, R22.2
- new net N$59: Q13.3, R28.2, R29.2, R30.2, R31.2, R32.2
- new net N$6: A2.A, R2.1
- new net N$60: Q13.1, R61.1, R62.2
- new net N$61: Q14.3, R62.1
- new net N$62: Q15.3, R33.2, R34.2, R35.2, R36.2, R37.2, R38.2
- new net N$63: Q15.1, R64.1, R65.2
- new net N$64: Q16.3, R65.1
- new net N$65: Q17.3, R39.2, R40.2, R41.2, R42.2
- new net N$66: Q17.1, R67.1, R68.2
- new net N$67: Q18.3, R68.1
- new net N$68: JP1.1, Q3.2, R47.2
- new net N$69: Q11.3, R23.2, R24.2, R25.2, R26.2, R27.2
- new net N$7: B1.A, R7.1
- new net N$8: B2.A, R8.1
- new net N$9: B3.A, R9.1
- net A: now also Q1.1, R43.2
- net B: now also Q6.1, R51.2
- net C: now also Q8.1, R54.2
- net D: now also Q10.1, R57.2
- net DOT: now also Q18.1, R69.2
- net E: now also Q12.1, R60.2
- net F: now also Q14.1, R63.2
- net G: now also Q16.1, R66.2
- net GND: now also Q1.2, Q10.2, Q12.2, Q14.2, Q16.2, Q18.2, Q4.2, Q6.2, Q8.2, R43.1, R48.1, R51.1, R54.1, R57.1, R60.1, R63.1, R66.1, R69.1
- net VCC: now also JP1.2, Q11.2, Q13.2, Q15.2, Q17.2, Q2.2, Q5.2, Q7.2, Q9.2, R44.2, R49.2, R52.2, R55.2, R58.2, R61.2, R64.2, R67.2
Routing:
- net COMMON: track 0.00 -> 427.5 mm, vias 0 -> 5
- net VCC: track 0.00 -> 312.5 mm, vias 0 -> 9
- net N$62: track 0.00 -> 58.6 mm, vias 0 -> 2
- net N$55: track 0.00 -> 58.5 mm, vias 0 -> 4
- net N$58: track 0.00 -> 54.8 mm
- net D: track 82.5 -> 133.3 mm, vias 0 -> 2
- net !ENABLE!: track 0.00 -> 50.7 mm, vias 0 -> 2
- net N$69: track 0.00 -> 49.9 mm, vias 0 -> 4
- net N$46: track 0.00 -> 49.3 mm
- net N$49: track 0.00 -> 46.1 mm, vias 0 -> 2
- net N$59: track 0.00 -> 45.8 mm, vias 0 -> 2
- net A: track 82.5 -> 120.0 mm, vias 0 -> 2
- net C: track 82.5 -> 118.0 mm, vias 0 -> 4
- net N$65: track 0.00 -> 32.1 mm, vias 0 -> 2
- net F: track 82.5 -> 114.3 mm, vias 0 -> 2
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Other:
- board text added: "!EN!"
- board text added: "-"
- board text added: "A"
- board text added: "B"
- board text added: "C"
- board text added: "D"
- board text added: "DOT"
- board text added: "E"
- board text added: "F"
- board text added: "G"
- board text added: "To make Enable pin Active HIGH"
- board text added: "cut JP1 and bridge JP2"
