File: big7segment with sec delimiter/big7segment.brd (EAGLE design)
At the start: 90 x 122 mm, 156 parts, among them Q1 NMOS, Q10 NMOS, Q11 PMOS, Q12 NMOS, Q13 PMOS, Q14 NMOS, Q15 PMOS, Q16 NMOS, Q17 PMOS, Q18 NMOS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

Commit message: big7segment with sec board layout
Parts:
- added -_SEC, -_SEC1, 5V_SEC, 5V_SEC1, GND_SEC, GND_SEC1, SEC: (no value), SparkFun-Connectors:1X01_OFFSET
- added LED1, LED2: (no value), led:LED5MM
- added Q19: NMOS, SparkFun-DiscreteSemi:SOT23-3
- added R70: 10k, SparkFun-Resistors:0805
- added R71, R72: 180, SparkFun-Resistors:0805
Connections:
- new net GND_SEC: -_SEC.1, -_SEC1.1, GND_SEC.1, GND_SEC1.1, Q19.2, R70.1
- new net N$70: LED2.A, R72.1
- new net N$71: LED1.A, R71.1
- new net N$75: LED1.K, LED2.K, Q19.3
- new net SEC: Q19.1, R70.2, SEC.1
- new net VCC_1: 5V_SEC.1, 5V_SEC1.1, R71.2, R72.2
Routing:
- net VCC_1: track 0.00 -> 66.4 mm
- net SEC: track 0.00 -> 65.9 mm
- net GND_SEC: track 0.00 -> 53.5 mm
- net N$75: track 0.00 -> 51.5 mm
- net N$70: track 0.00 -> 5.27 mm
- net N$71: track 0.00 -> 5.08 mm
Other:
- board size 90 x 122 mm -> 123.8 x 122 mm
Changed lines of the file:
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@@
 <text x="53.975" y="28.8925" size="1.016" layer="26" font="vector" rot="MR0">cut JP1 and bridge JP2</text>
 <text x="84.455" y="25.4" size="0.762" layer="25" font="vector" ratio="13" rot="R90" align="bottom-center">-</text>
+<wire x1="120.015" y1="121.92" x2="107.315" y2="121.92" width="0.2032" layer="20"/>
+<wire x1="107.315" y1="121.92" x2="103.505" y2="118.11" width="0.2032" layer="20" curve="90"/>
+<wire x1="103.505" y1="3.81" x2="107.315" y2="0" width="0.2032" layer="20" curve="90"/>
+<wire x1="107.315" y1="0" x2="120.015" y2="0" width="0.2032" layer="20"/>
+<wire x1="120.015" y1="0" x2="123.825" y2="3.81" width="0.2032" layer="20" curve="90"/>
+<wire x1="123.825" y1="3.81" x2="123.825" y2="118.11" width="0.2032" layer="20"/>
+<wire x1="123.825" y1="118.11" x2="120.015" y2="121.92" width="0.2032" layer="20" curve="90"/>
+<wire x1="103.505" y1="3.81" x2="103.505" y2="118.11" width="0.2032" layer="20"/>
+<hole x="113.66" y="118" drill="3.2"/>
+<hole x="113.6" y="4" drill="3.2"/>
 </plain>
 <attributes>
@@
 </element>
 <element name="JP2" library="SparkFun-Jumpers" package="SMT-JUMPER_2_NO_NO-SILK" value="" x="40.3225" y="35.2425" rot="MR180"/>
+<element name="SEC" library="SparkFun-Connectors" package="1X01_OFFSET" value="" x="114.3" y="17.78" rot="R90"/>
+<element name="5V_SEC" library="SparkFun-Connectors" package="1X01_OFFSET" value="" x="116.84" y="27.94" smashed="yes" rot="R90">
+<attribute name="VALUE" x="118.872" y="26.67" size="0.6096" layer="27" font="vector" ratio="20" rot="R90"/>
+</element>
+<element name="-_SEC" library="SparkFun-Connectors" package="1X01_OFFSET" value="" x="116.84" y="25.4" smashed="yes" rot="R90">
+<attribute name="VALUE" x="118.872" y="24.13" size="0.6096" layer="27" font="vector" ratio="20" rot="R90"/>
+</element>
+<element name="GND_SEC" library="SparkFun-Connectors" package="1X01_OFFSET" value="" x="116.84" y="22.86" smashed="yes" rot="R90">
+<attribute name="VALUE" x="118.872" y="21.59" size="0.6096" layer="27" font="vector" ratio="20" rot="R90"/>
+</element>
+<element name="Q19" library="SparkFun-DiscreteSemi" package="SOT23-3" value="NMOS" x="113.9825" y="60.96" rot="MR0">
+<attribute name="PROD_ID" value="TRANS-12988" x="113.9825" y="60.96" size="1.778" layer="28" rot="MR0" display="off"/>
+</element>
+<element name="R70" library="SparkFun-Resistors" package="0805" value="10k" x="113.665" y="56.515" rot="MR180">
+<attribute name="PROD_ID" value="RES-11622" x="113.665" y="56.515" size="1.778" layer="28" rot="MR180" display="off"/>
+</element>
+<element name="R71" library="SparkFun-Resistors" package="0805" value="180" x="115.57" y="78.74" rot="MR0">
+<attribute name="PROD_ID" value="RES-11622" x="119.0625" y="74.93" size="1.778" layer="28" rot="MR0" display="off"/>
+</element>
+<element name="R72" library="SparkFun-Resistors" package="0805" value="180" x="107.95" y="33.02" rot="MR0">
+<attribute name="PROD_ID" value="RES-11622" x="107.6325" y="29.21" size="1.778" layer="28" rot="MR0" display="off"/>
+</element>
+<element name="LED1" library="led" package="LED5MM" value="" x="117.729" y="83.82"/>
+<element name="LED2" library="led" package="LED5MM" value="" x="109.6645" y="38.1"/>
+<element name="5V_SEC1" library="SparkFun-Connectors" package="1X01_OFFSET" value="" x="111.76" y="27.94" smashed="yes" rot="R90">
+<attribute name="VALUE" x="113.792" y="26.67" size="0.6096" layer="27" font="vector" ratio="20" rot="R90"/>
+</element>
+<element name="-_SEC1" library="SparkFun-Connectors" package="1X01_OFFSET" value="" x="111.76" y="25.4" smashed="yes" rot="R90">
+<attribute name="VALUE" x="113.792" y="24.13" size="0.6096" layer="27" font="vector" ratio="20" rot="R90"/>
+</element>
+<element name="GND_SEC1" library="SparkFun-Connectors" package="1X01_OFFSET" value="" x="111.76" y="22.86" smashed="yes" rot="R90">
+<attribute name="VALUE" x="113.792" y="21.59" size="0.6096" layer="27" font="vector" ratio="20" rot="R90"/>
+</element>
 </elements>
 <signals>
@@
 <wire x1="44.1325" y1="37.592" x2="47.31" y2="33.29" width="0.2032" layer="16"/>
 </signal>
+<signal name="N$75">
+<contactref element="Q19" pad="3"/>
+<contactref element="LED1" pad="K"/>
+<contactref element="LED2" pad="K"/>
+<wire x1="118.999" y1="83.82" x2="118.999" y2="67.0765" width="0.8128" layer="16"/>
+<wire x1="118.999" y1="67.0765" x2="113.9825" y2="62.06" width="0.8128" layer="16"/>
+<wire x1="113.9825" y1="62.06" x2="111.59" y2="62.06" width="0.8128" layer="16"/>
+<wire x1="111.59" y1="62.06" x2="109.855" y2="60.325" width="0.8128" layer="16"/>
+<wire x1="109.855" y1="60.325" x2="109.855" y2="46.355" width="0.8128" layer="16"/>
+<wire x1="109.855" y1="46.355" x2="111.125" y2="45.085" width="0.8128" layer="16"/>
+<wire x1="111.125" y1="45.085" x2="111.125" y2="38.2905" width="0.8128" layer="16"/>
+<wire x1="111.125" y1="38.2905" x2="110.9345" y2="38.1" width="0.8128" layer="16"/>
+</signal>
+<signal name="SEC">
+<contactref element="SEC" pad="1"/>
+<contactref element="Q19" pad="1"/>
+<contactref element="R70" pad="2"/>
+<wire x1="114.9325" y1="59.96" x2="114.9325" y2="56.8825" width="0.8128" layer="16"/>
+<wire x1="114.9325" y1="56.8825" x2="114.565" y2="56.515" width="0.4064" layer="16"/>
+<wire x1="114.3" y1="17.78" x2="116.84" y2="17.78" width="0.8128" layer="16"/>
+<wire x1="116.84" y1="17.78" x2="116.84" y2="19.685" width="0.8128" layer="16"/>
+<wire x1="116.84" y1="19.685" x2="113.03" y2="19.685" width="0.8128" layer="16"/>
+<wire x1="113.03" y1="19.685" x2="113.03" y2="15.875" width="0.8128" layer="16"/>
+<wire x1="113.03" y1="15.875" x2="116.84" y2="15.875" width="0.8128" layer="16"/>
+<wire x1="116.84" y1="15.875" x2="116.84" y2="17.78" width="0.8128" layer="16"/>
+<wire x1="116.84" y1="17.78" x2="118.745" y2="17.78" width="0.8128" layer="16"/>
+<wire x1="118.745" y1="17.78" x2="121.285" y2="20.32" width="0.8128" layer="16"/>
+<wire x1="121.285" y1="20.32" x2="121.285" y2="46.99" width="0.8128" layer="16"/>
+<wire x1="121.285" y1="46.99" x2="114.935" y2="53.34" width="0.8128" layer="16"/>
+<wire x1="114.935" y1="53.34" x2="114.935" y2="56.145" width="0.8128" layer="16"/>
+<wire x1="114.935" y1="56.145" x2="114.565" y2="56.515" width="0.8128" layer="16"/>
+</signal>
+<signal name="VCC_1">
+<contactref element="R71" pad="2"/>
+<contactref element="R72" pad="2"/>
+<contactref element="5V_SEC" pad="1"/>
+<wire x1="114.67" y1="78.74" x2="114.67" y2="70.22" width="0.8128" layer="16"/>
+<wire x1="114.67" y1="70.22" x2="105.41" y2="60.96" width="0.8128" layer="16"/>
+<wire x1="105.41" y1="60.96" x2="105.41" y2="34.66" width="0.8128" layer="16"/>
+<wire x1="105.41" y1="34.66" x2="105.595" y2="34.475" width="0.8128" layer="16"/>
+<contactref element="5V_SEC1" pad="1"/>
+<wire x1="105.595" y1="34.475" x2="107.05" y2="33.02" width="0.8128" layer="16"/>
+<wire x1="111.76" y1="27.94" x2="108.585" y2="27.94" width="0.8128" layer="16"/>
+<wire x1="108.585" y1="27.94" x2="105.41" y2="31.115" width="0.8128" layer="16"/>
+<wire x1="105.41" y1="31.115" x2="105.41" y2="34.29" width="0.8128" layer="16"/>
+<wire x1="105.41" y1="34.29" x2="105.595" y2="34.475" width="0.8128" layer="16"/>
+<wire x1="116.84" y1="27.94" x2="111.76" y2="27.94" width="0.8128" layer="16"/>
+</signal>
+<signal name="GND_SEC">
+<contactref element="GND_SEC" pad="1"/>
+<contactref element="-_SEC" pad="1"/>
+<contactref element="Q19" pad="2"/>
+<contactref element="R70" pad="1"/>
+<wire x1="113.0325" y1="59.96" x2="113.0325" y2="56.7825" width="0.8128" layer="16"/>
+<wire x1="113.0325" y1="56.7825" x2="112.765" y2="56.515" width="0.4064" layer="16"/>
+<wire x1="116.84" y1="25.4" x2="116.84" y2="22.86" width="0.8128" layer="16"/>
+<contactref element="-_SEC1" pad="1"/>
+<contactref element="GND_SEC1" pad="1"/>
+<wire x1="111.76" y1="22.86" x2="111.76" y2="25.4" width="0.8128" layer="16"/>
+<wire x1="111.76" y1="25.4" x2="116.84" y2="25.4" width="0.8128" layer="16"/>
+<wire x1="111.76" y1="25.4" x2="117.475" y2="25.4" width="0.8128" layer="16"/>
+<wire x1="117.475" y1="25.4" x2="118.745" y2="26.67" width="0.8128" layer="16"/>
+<wire x1="118.745" y1="26.67" x2="118.745" y2="46.355" width="0.8128" layer="16"/>
+<wire x1="118.745" y1="46.355" x2="113.03" y2="52.07" width="0.8128" layer="16"/>
+<wire x1="113.03" y1="52.07" x2="113.03" y2="56.25" width="0.8128" layer="16"/>
+<wire x1="113.03" y1="56.25" x2="112.765" y2="56.515" width="0.8128" layer="16"/>
+</signal>
+<signal name="N$70">
+<contactref element="LED2" pad="A"/>
+<contactref element="R72" pad="1"/>
+<wire x1="108.85" y1="33.02" x2="108.85" y2="37.6445" width="0.8128" layer="16"/>
+<wire x1="108.85" y1="37.6445" x2="108.3945" y2="38.1" width="0.8128" layer="16"/>
+</signal>
+<signal name="N$71">
+<contactref element="LED1" pad="A"/>
+<contactref element="R71" pad="1"/>
+<wire x1="116.47" y1="78.74" x2="116.47" y2="83.809" width="0.8128" layer="16"/>
+<wire x1="116.47" y1="83.809" x2="116.459" y2="83.82" width="0.4064" layer="16"/>
+</signal>
 </signals>
